File: ChemE/ChemE.kicad_pcb (KiCad board)
At the start: 2 copper layers, 36 x 26 mm, 12 parts, among them IC1 LF353P, Q1 MTP3055E, U1 LM393N

Commit message: added my name. ordered
Other:
- board text added: "Made by Caleb Murray"
Changed lines of the file:
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@@
+		)
+	)
+	(gr_text "Made by Caleb Murray"
+		(at 179.1716 115.0112 -0)
+		(layer "B.SilkS")
+		(effects
+			(font
+				(size 1.5 1.5)
+				(thickness 0.3)
+				(bold yes)
+			)
+			(justify left bottom mirror)
 		)
 	)

Commit message: updated design w/ new components and footprints
Parts:
- removed Pot: 10k pot, Potentiometer_THT:Potentiometer_Piher_PT-6-H_Horizontal
- removed Q1: MTP3055E, Package_TO_SOT_THT:TO-247-3_Vertical
- added Q**: TO254P469X1042X1967-3P, mosfet:TO254P469X1042X1967-3P, F.Cu at (193.2, 110.1)
- added REF**: POT_3296W, step:POT_3296W, F.Cu at (193.0, 114.8)
- renumbered +9V to J1

Commit message: ordered and closed
Parts:
- removed Q**: TO254P469X1042X1967-3P, mosfet:TO254P469X1042X1967-3P
- removed REF**: POT_3296W, step:POT_3296W
- added Q2: IRLZ44NPBF, mosfet:TO254P469X1042X1967-3P, F.Cu at (183.3, 117.1)
- added R4: 3296W-1-103LF, step:POT_3296W, F.Cu at (153.5, 116.5)
Routing:
- net GND: track 7.80 -> 0.04 mm
- net Net-(D2-A): track 13.8 -> 20.0 mm
- net +9V: track 33.4 -> 39.5 mm
- net Net-(U1-NEG_A): track 12.6 -> 14.6 mm
- net Net-(Q2-G): track 10.7 -> 12.0 mm
